Commit message: add first maze

File: description/robot_core.xacro (robot description, xacro)
@@ -2,4 +2,5 @@
 <robot xmlns:xacro="http://www.ros.org/wiki/xacro">
     <xacro:include filename="inertial_macros.xacro"/>
+    <xacro:include filename="gazebo_control.xacro"/>
     <material name="white">
         <color rgba="1 1 1 1" />
@@ -39,4 +40,7 @@
         </xacro:inertial_box>
     </link>
+    <gazebo reference="chassis">
+        <material>Gazebo/White</material>
+    </gazebo>
     <joint name="left_wheel_joint" type="continuous">
         <parent link="base_link"/>
@@ -61,4 +65,7 @@
         </xacro:inertial_cylinder>
     </link>
+    <gazebo reference="left_wheel">
+        <material>Gazebo/Blue</material>
+    </gazebo>
      <joint name="right_wheel_joint" type="continuous">
         <parent link="base_link"/>
@@ -83,4 +90,7 @@
         </xacro:inertial_cylinder>
     </link>
+    <gazebo reference="right_wheel">
+        <material>Gazebo/Blue</material>
+    </gazebo>
     <joint name="caster_wheel_joint" type="fixed">
         <parent link="chassis"/>
@@ -104,3 +114,8 @@
         </xacro:inertial_sphere>
     </link>
+    <gazebo reference="caster_wheel">
+        <material>Gazebo/Black</material>
+        <mu1 value="0.001"/>
+        <mu2 value="0.001"/>
+    </gazebo>
 </robot>

Commit message: add lidar on robot

File: description/robot_core.xacro (robot description, xacro)
@@ -15,5 +15,8 @@
         <color rgba="0 0 0 1"/>
     </material>
-     <link name="base_link">
+    <material name="red">
+        <color rgba="1 0 0 1"/>
+    </material>
+    <link name="base_link">
     </link>
     <joint name="chassis_joint" type="fixed">
